File: DIO_FATAR/DIO_FATAR.kicad_pcb (KiCad board)
At the start: 2 copper layers, 100 x 50 mm, 20 parts, among them J1 in, J2 thru, J3 right, J4 left, U1 74HC595, U2 74HC595, U3 74165, U4 74165

Commit message: DIO_FATAR: remove mounting hole references
Parts:
- renumbered REF** to ?
Changed lines of the file:
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@@
     (tags "mounting hole 3.2mm no annular m3 din965")
     (attr virtual)
-    (fp_text reference REF** (at 0 -3.8) (layer F.SilkS)
+    (fp_text reference "" (at 0 -3.8) (layer F.SilkS)
       (effects (font (size 1 1) (thickness 0.15)))
     )
@@
     (tags "mounting hole 3.2mm no annular m3 din965")
     (attr virtual)
-    (fp_text reference REF** (at 0 -3.8) (layer F.SilkS)
+    (fp_text reference "" (at 0 -3.8) (layer F.SilkS)
       (effects (font (size 1 1) (thickness 0.15)))
     )
@@
     (tags "mounting hole 3.2mm no annular m3 din965")
     (attr virtual)
-    (fp_text reference REF** (at 0 -3.8) (layer F.SilkS)
+    (fp_text reference "" (at 0 -4.39) (layer F.SilkS)
       (effects (font (size 1 1) (thickness 0.15)))
     )
@@
     (tags "mounting hole 3.2mm no annular m3 din965")
     (attr virtual)
-    (fp_text reference REF** (at 0 -3.8) (layer F.SilkS)
+    (fp_text reference "" (at 0 -3.8) (layer F.SilkS)
       (effects (font (size 1 1) (thickness 0.15)))
     )
